Commit message: Update hithand_to_mujoco.urdf

File: hithand_to_mujoco.urdf (robot description, URDF)
Before this commit: robot hithand, 22 links, 21 joints
Links:
- link Right_Index_Basecover: geometry collision mesh filename=meshes/hit-hand-2-finger-basecover.stl; visual mesh filename=meshes/hit-hand-2-finger-basecover.stl
- link Right_Index_Phadist: geometry collision mesh filename=meshes/hit-hand-2-finger-phadist.stl; visual mesh filename=meshes/hit-hand-2-finger-phadist.stl
- link Right_Index_Phamed: geometry collision mesh filename=meshes/hit-hand-2-finger-phamed.stl; visual mesh filename=meshes/hit-hand-2-finger-phamed.stl
- link Right_Index_Phoaprox: geometry collision mesh filename=meshes/hit-hand-2-finger-phaprox.stl; visual mesh filename=meshes/hit-hand-2-finger-phaprox.stl
- link Right_Little_Basecover: geometry collision mesh filename=meshes/hit-hand-2-finger-basecover.stl; visual mesh filename=meshes/hit-hand-2-finger-basecover.stl
- link Right_Little_Phadist: geometry collision mesh filename=meshes/hit-hand-2-finger-phadist.stl; visual mesh filename=meshes/hit-hand-2-finger-phadist.stl
- link Right_Little_Phamed: geometry collision mesh filename=meshes/hit-hand-2-finger-phamed.stl; visual mesh filename=meshes/hit-hand-2-finger-phamed.stl
- link Right_Little_Phoaprox: geometry collision mesh filename=meshes/hit-hand-2-finger-phaprox.stl; visual mesh filename=meshes/hit-hand-2-finger-phaprox.stl
- link Right_Middle_Basecover: geometry collision mesh filename=meshes/hit-hand-2-finger-basecover.stl; visual mesh filename=meshes/hit-hand-2-finger-basecover.stl
- link Right_Middle_Phadist: geometry collision mesh filename=meshes/hit-hand-2-finger-phadist.stl; visual mesh filename=meshes/hit-hand-2-finger-phadist.stl
- link Right_Middle_Phamed: geometry collision mesh filename=meshes/hit-hand-2-finger-phamed.stl; visual mesh filename=meshes/hit-hand-2-finger-phamed.stl
- link Right_Middle_Phoaprox: geometry collision mesh filename=meshes/hit-hand-2-finger-phaprox.stl; visual mesh filename=meshes/hit-hand-2-finger-phaprox.stl
- link Right_Ring_Basecover: geometry collision mesh filename=meshes/hit-hand-2-finger-basecover.stl; visual mesh filename=meshes/hit-hand-2-finger-basecover.stl
- link Right_Ring_Phadist: geometry collision mesh filename=meshes/hit-hand-2-finger-phadist.stl; visual mesh filename=meshes/hit-hand-2-finger-phadist.stl
- link Right_Ring_Phamed: geometry collision mesh filename=meshes/hit-hand-2-finger-phamed.stl; visual mesh filename=meshes/hit-hand-2-finger-phamed.stl
- link Right_Ring_Phoaprox: geometry collision mesh filename=meshes/hit-hand-2-finger-phaprox.stl; visual mesh filename=meshes/hit-hand-2-finger-phaprox.stl
- link Right_Thumb_Basecover: geometry collision mesh filename=meshes/hit-hand-2-finger-basecover.stl; visual mesh filename=meshes/hit-hand-2-finger-basecover.stl
- link Right_Thumb_Phadist: geometry collision mesh filename=meshes/hit-hand-2-finger-phadist.stl; visual mesh filename=meshes/hit-hand-2-finger-phadist.stl
- link Right_Thumb_Phamed: geometry collision mesh filename=meshes/hit-hand-2-finger-phamed.stl; visual mesh filename=meshes/hit-hand-2-finger-phamed.stl
- link Right_Thumb_Phoaprox: geometry collision mesh filename=meshes/hit-hand-2-finger-phaprox.stl; visual mesh filename=meshes/hit-hand-2-finger-phaprox.stl
- link base_link: geometry collision mesh filename=meshes/hit-hand-2-palm-right.stl; visual mesh filename=meshes/hit-hand-2-palm-right.stl
